Commit message: launch 4 robots added

File: ros2_mecademic_bringup/urdf/meca_500_r3_1.urdf (robot description, URDF)
Before this commit: robot meca_500_r3, 7 links, 6 joints
Links:
- removed link meca_axis_1_link
- removed link meca_axis_2_link
- removed link meca_axis_3_link
- removed link meca_axis_4_link
- removed link meca_axis_5_link
- removed link meca_axis_6_link
- removed link meca_base_link
- added link robot1/meca_axis_1_link; collision mesh filename=package://ros2_mecademic_description/meshes/meca_500_r3_j1_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; visual mesh filename=package://ros2_mecademic_description/meshes/meca_500_r3_j1.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
- added link robot1/meca_axis_2_link; collision mesh filename=package://ros2_mecademic_description/meshes/meca_500_r3_j2_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; visual mesh filename=package://ros2_mecademic_description/meshes/meca_500_r3_j2.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
- added link robot1/meca_axis_3_link; collision mesh filename=package://ros2_mecademic_description/meshes/meca_500_r3_j3_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; visual mesh filename=package://ros2_mecademic_description/meshes/meca_500_r3_j3.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
- added link robot1/meca_axis_4_link; collision mesh filename=package://ros2_mecademic_description/meshes/meca_500_r3_j4_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; visual mesh filename=package://ros2_mecademic_description/meshes/meca_500_r3_j4.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
- added link robot1/meca_axis_5_link; collision mesh filename=package://ros2_mecademic_description/meshes/meca_500_r3_j5_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; visual mesh filename=package://ros2_mecademic_description/meshes/meca_500_r3_j5.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
- added link robot1/meca_axis_6_link; collision mesh filename=package://ros2_mecademic_description/meshes/meca_500_r3_j6_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; visual mesh filename=package://ros2_mecademic_description/meshes/meca_500_r3_j6.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
- added link robot1/meca_base_link; collision mesh filename=package://ros2_mecademic_description/meshes/meca_500_r3_bas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; visual mesh filename=package://ros2_mecademic_description/meshes/meca_500_r3_bas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
- added link world
Joints:
- removed joint meca_axis_1_joint
- removed joint meca_axis_2_joint
- removed joint meca_axis_3_joint
- removed joint meca_axis_4_joint
- removed joint meca_axis_5_joint
- removed joint meca_axis_6_joint
- added joint robot1/meca_axis_1_joint: type revolute, parent robot1/meca_base_link, child robot1/meca_axis_1_link, origin xyz=0.012498 0 0.091 rpy=0 0 0, axis 0 0 1, limit lower=-3.05433 upper=3.05433 effort=10.0 velocity=2.61799
- added joint robot1/meca_axis_2_joint: type revolute, parent robot1/meca_axis_1_link, child robot1/meca_axis_2_link, origin xyz=0 0 0.044 rpy=0 0 0, axis 0 1 0, limit lower=-1.22173048 upper=1.5708 effort=10.0 velocity=2.61799
- added joint robot1/meca_axis_3_joint: type revolute, parent robot1/meca_axis_2_link, child robot1/meca_axis_3_link, origin xyz=0 0 0.135 rpy=0 0 0, axis 0 1 0, limit lower=-2.35619 upper=1.22173048 effort=10.0 velocity=3.14159
- added joint robot1/meca_axis_4_joint: type revolute, parent robot1/meca_axis_3_link, child robot1/meca_axis_4_link, origin xyz=0 0 0.038 rpy=0 0 0, axis 1 0 0, limit lower=-2.96706 upper=2.96706 effort=10.0 velocity=5.23599
- added joint robot1/meca_axis_5_joint: type revolute, parent robot1/meca_axis_4_link, child robot1/meca_axis_5_link, origin xyz=0.12 0 0 rpy=0 0 0, axis 0 1 0, limit lower=-2.00713 upper=2.00713 effort=10.0 velocity=5.23599
- added joint robot1/meca_axis_6_joint: type revolute, parent robot1/meca_axis_5_link, child robot1/meca_axis_6_link, origin xyz=0.07 0 0 rpy=0 0 0, axis 1 0 0, limit lower=-3.14159 upper=3.14159 effort=10.0 velocity=8.72665
- added joint robot1/world_joint: type fixed, parent world, child robot1/meca_base_link, origin xyz=0.5 0.5 0 rpy=0 0 0, axis 0 0 0

File: ros2_mecademic_bringup/urdf/meca_500_r3_2.urdf (robot description, URDF)
Before this commit: robot meca_500_r3, 7 links, 6 joints
Links:
- removed link meca_axis_1_link
- removed link meca_axis_2_link
- removed link meca_axis_3_link
- removed link meca_axis_4_link
- removed link meca_axis_5_link
- removed link meca_axis_6_link
- removed link meca_base_link
- added link robot2/meca_axis_1_link; collision mesh filename=package://ros2_mecademic_description/meshes/meca_500_r3_j1_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; visual mesh filename=package://ros2_mecademic_description/meshes/meca_500_r3_j1.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
- added link robot2/meca_axis_2_link; collision mesh filename=package://ros2_mecademic_description/meshes/meca_500_r3_j2_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; visual mesh filename=package://ros2_mecademic_description/meshes/meca_500_r3_j2.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
- added link robot2/meca_axis_3_link; collision mesh filename=package://ros2_mecademic_description/meshes/meca_500_r3_j3_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; visual mesh filename=package://ros2_mecademic_description/meshes/meca_500_r3_j3.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
- added link robot2/meca_axis_4_link; collision mesh filename=package://ros2_mecademic_description/meshes/meca_500_r3_j4_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; visual mesh filename=package://ros2_mecademic_description/meshes/meca_500_r3_j4.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
- added link robot2/meca_axis_5_link; collision mesh filename=package://ros2_mecademic_description/meshes/meca_500_r3_j5_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; visual mesh filename=package://ros2_mecademic_description/meshes/meca_500_r3_j5.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
- added link robot2/meca_axis_6_link; collision mesh filename=package://ros2_mecademic_description/meshes/meca_500_r3_j6_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; visual mesh filename=package://ros2_mecademic_description/meshes/meca_500_r3_j6.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
- added link robot2/meca_base_link; collision mesh filename=package://ros2_mecademic_description/meshes/meca_500_r3_bas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; visual mesh filename=package://ros2_mecademic_description/meshes/meca_500_r3_bas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
- added link world
Joints:
- removed joint meca_axis_1_joint
- removed joint meca_axis_2_joint
- removed joint meca_axis_3_joint
- removed joint meca_axis_4_joint
- removed joint meca_axis_5_joint
- removed joint meca_axis_6_joint
- added joint robot2/meca_axis_1_joint: type revolute, parent robot2/meca_base_link, child robot2/meca_axis_1_link, origin xyz=0.012498 0 0.091 rpy=0 0 0, axis 0 0 1, limit lower=-3.05433 upper=3.05433 effort=10.0 velocity=2.61799
- added joint robot2/meca_axis_2_joint: type revolute, parent robot2/meca_axis_1_link, child robot2/meca_axis_2_link, origin xyz=0 0 0.044 rpy=0 0 0, axis 0 1 0, limit lower=-1.22173048 upper=1.5708 effort=10.0 velocity=2.61799
- added joint robot2/meca_axis_3_joint: type revolute, parent robot2/meca_axis_2_link, child robot2/meca_axis_3_link, origin xyz=0 0 0.135 rpy=0 0 0, axis 0 1 0, limit lower=-2.35619 upper=1.22173048 effort=10.0 velocity=3.14159
- added joint robot2/meca_axis_4_joint: type revolute, parent robot2/meca_axis_3_link, child robot2/meca_axis_4_link, origin xyz=0 0 0.038 rpy=0 0 0, axis 1 0 0, limit lower=-2.96706 upper=2.96706 effort=10.0 velocity=5.23599
- added joint robot2/meca_axis_5_joint: type revolute, parent robot2/meca_axis_4_link, child robot2/meca_axis_5_link, origin xyz=0.12 0 0 rpy=0 0 0, axis 0 1 0, limit lower=-2.00713 upper=2.00713 effort=10.0 velocity=5.23599
- added joint robot2/meca_axis_6_joint: type revolute, parent robot2/meca_axis_5_link, child robot2/meca_axis_6_link, origin xyz=0.07 0 0 rpy=0 0 0, axis 1 0 0, limit lower=-3.14159 upper=3.14159 effort=10.0 velocity=8.72665
- added joint robot2/world_joint: type fixed, parent world, child robot2/meca_base_link, origin xyz=0.5 -0.5 0 rpy=0 0 0, axis 0 0 0

File: ros2_mecademic_bringup/urdf/meca_500_r3_3.urdf (robot description, URDF)
Before this commit: robot meca_500_r3, 7 links, 6 joints
Links:
- removed link meca_axis_1_link
- removed link meca_axis_2_link
- removed link meca_axis_3_link
- removed link meca_axis_4_link
- removed link meca_axis_5_link
- removed link meca_axis_6_link
- removed link meca_base_link
- added link robot3/meca_axis_1_link; collision mesh filename=package://ros2_mecademic_description/meshes/meca_500_r3_j1_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; visual mesh filename=package://ros2_mecademic_description/meshes/meca_500_r3_j1.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
- added link robot3/meca_axis_2_link; collision mesh filename=package://ros2_mecademic_description/meshes/meca_500_r3_j2_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; visual mesh filename=package://ros2_mecademic_description/meshes/meca_500_r3_j2.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
- added link robot3/meca_axis_3_link; collision mesh filename=package://ros2_mecademic_description/meshes/meca_500_r3_j3_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; visual mesh filename=package://ros2_mecademic_description/meshes/meca_500_r3_j3.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
- added link robot3/meca_axis_4_link; collision mesh filename=package://ros2_mecademic_description/meshes/meca_500_r3_j4_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; visual mesh filename=package://ros2_mecademic_description/meshes/meca_500_r3_j4.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
- added link robot3/meca_axis_5_link; collision mesh filename=package://ros2_mecademic_description/meshes/meca_500_r3_j5_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; visual mesh filename=package://ros2_mecademic_description/meshes/meca_500_r3_j5.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
- added link robot3/meca_axis_6_link; collision mesh filename=package://ros2_mecademic_description/meshes/meca_500_r3_j6_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; visual mesh filename=package://ros2_mecademic_description/meshes/meca_500_r3_j6.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
- added link robot3/meca_base_link; collision mesh filename=package://ros2_mecademic_description/meshes/meca_500_r3_bas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; visual mesh filename=package://ros2_mecademic_description/meshes/meca_500_r3_bas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
- added link world
Joints:
- removed joint meca_axis_1_joint
- removed joint meca_axis_2_joint
- removed joint meca_axis_3_joint
- removed joint meca_axis_4_joint
- removed joint meca_axis_5_joint
- removed joint meca_axis_6_joint
- added joint robot3/meca_axis_1_joint: type revolute, parent robot3/meca_base_link, child robot3/meca_axis_1_link, origin xyz=0.012498 0 0.091 rpy=0 0 0, axis 0 0 1, limit lower=-3.05433 upper=3.05433 effort=10.0 velocity=2.61799
- added joint robot3/meca_axis_2_joint: type revolute, parent robot3/meca_axis_1_link, child robot3/meca_axis_2_link, origin xyz=0 0 0.044 rpy=0 0 0, axis 0 1 0, limit lower=-1.22173048 upper=1.5708 effort=10.0 velocity=2.61799
- added joint robot3/meca_axis_3_joint: type revolute, parent robot3/meca_axis_2_link, child robot3/meca_axis_3_link, origin xyz=0 0 0.135 rpy=0 0 0, axis 0 1 0, limit lower=-2.35619 upper=1.22173048 effort=10.0 velocity=3.14159
- added joint robot3/meca_axis_4_joint: type revolute, parent robot3/meca_axis_3_link, child robot3/meca_axis_4_link, origin xyz=0 0 0.038 rpy=0 0 0, axis 1 0 0, limit lower=-2.96706 upper=2.96706 effort=10.0 velocity=5.23599
- added joint robot3/meca_axis_5_joint: type revolute, parent robot3/meca_axis_4_link, child robot3/meca_axis_5_link, origin xyz=0.12 0 0 rpy=0 0 0, axis 0 1 0, limit lower=-2.00713 upper=2.00713 effort=10.0 velocity=5.23599
- added joint robot3/meca_axis_6_joint: type revolute, parent robot3/meca_axis_5_link, child robot3/meca_axis_6_link, origin xyz=0.07 0 0 rpy=0 0 0, axis 1 0 0, limit lower=-3.14159 upper=3.14159 effort=10.0 velocity=8.72665
- added joint robot3/world_joint: type fixed, parent world, child robot3/meca_base_link, origin xyz=-0.5 0.5 0 rpy=0 0 0, axis 0 0 0

File: ros2_mecademic_bringup/urdf/meca_500_r3_4.urdf (robot description, URDF)
Before this commit: robot meca_500_r3, 7 links, 6 joints
Links:
- removed link meca_axis_1_link
- removed link meca_axis_2_link
- removed link meca_axis_3_link
- removed link meca_axis_4_link
- removed link meca_axis_5_link
- removed link meca_axis_6_link
- removed link meca_base_link
- added link robot4/meca_axis_1_link; collision mesh filename=package://ros2_mecademic_description/meshes/meca_500_r3_j1_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; visual mesh filename=package://ros2_mecademic_description/meshes/meca_500_r3_j1.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
- added link robot4/meca_axis_2_link; collision mesh filename=package://ros2_mecademic_description/meshes/meca_500_r3_j2_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; visual mesh filename=package://ros2_mecademic_description/meshes/meca_500_r3_j2.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
- added link robot4/meca_axis_3_link; collision mesh filename=package://ros2_mecademic_description/meshes/meca_500_r3_j3_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; visual mesh filename=package://ros2_mecademic_description/meshes/meca_500_r3_j3.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
- added link robot4/meca_axis_4_link; collision mesh filename=package://ros2_mecademic_description/meshes/meca_500_r3_j4_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; visual mesh filename=package://ros2_mecademic_description/meshes/meca_500_r3_j4.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
- added link robot4/meca_axis_5_link; collision mesh filename=package://ros2_mecademic_description/meshes/meca_500_r3_j5_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; visual mesh filename=package://ros2_mecademic_description/meshes/meca_500_r3_j5.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
- added link robot4/meca_axis_6_link; collision mesh filename=package://ros2_mecademic_description/meshes/meca_500_r3_j6_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; visual mesh filename=package://ros2_mecademic_description/meshes/meca_500_r3_j6.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
- added link robot4/meca_base_link; collision mesh filename=package://ros2_mecademic_description/meshes/meca_500_r3_bas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; visual mesh filename=package://ros2_mecademic_description/meshes/meca_500_r3_bas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
- added link world
Joints:
- removed joint meca_axis_1_joint
- removed joint meca_axis_2_joint
- removed joint meca_axis_3_joint
- removed joint meca_axis_4_joint
- removed joint meca_axis_5_joint
- removed joint meca_axis_6_joint
- added joint robot4/meca_axis_1_joint: type revolute, parent robot4/meca_base_link, child robot4/meca_axis_1_link, origin xyz=0.012498 0 0.091 rpy=0 0 0, axis 0 0 1, limit lower=-3.05433 upper=3.05433 effort=10.0 velocity=2.61799
- added joint robot4/meca_axis_2_joint: type revolute, parent robot4/meca_axis_1_link, child robot4/meca_axis_2_link, origin xyz=0 0 0.044 rpy=0 0 0, axis 0 1 0, limit lower=-1.22173048 upper=1.5708 effort=10.0 velocity=2.61799
- added joint robot4/meca_axis_3_joint: type revolute, parent robot4/meca_axis_2_link, child robot4/meca_axis_3_link, origin xyz=0 0 0.135 rpy=0 0 0, axis 0 1 0, limit lower=-2.35619 upper=1.22173048 effort=10.0 velocity=3.14159
- added joint robot4/meca_axis_4_joint: type revolute, parent robot4/meca_axis_3_link, child robot4/meca_axis_4_link, origin xyz=0 0 0.038 rpy=0 0 0, axis 1 0 0, limit lower=-2.96706 upper=2.96706 effort=10.0 velocity=5.23599
- added joint robot4/meca_axis_5_joint: type revolute, parent robot4/meca_axis_4_link, child robot4/meca_axis_5_link, origin xyz=0.12 0 0 rpy=0 0 0, axis 0 1 0, limit lower=-2.00713 upper=2.00713 effort=10.0 velocity=5.23599
- added joint robot4/meca_axis_6_joint: type revolute, parent robot4/meca_axis_5_link, child robot4/meca_axis_6_link, origin xyz=0.07 0 0 rpy=0 0 0, axis 1 0 0, limit lower=-3.14159 upper=3.14159 effort=10.0 velocity=8.72665
- added joint robot4/world_joint: type fixed, parent world, child robot4/meca_base_link, origin xyz=-0.5 -0.5 0 rpy=0 0 0, axis 0 0 0
